File: output_folder/pcbs/praline_uni.kicad_pcb (KiCad board)
At the start: 2 copper layers, 269.4 x 128.8 mm, 76 parts

Commit message: add routed pcbs
Parts:
- added G***: LOGO, LOGO, F.Cu at (197.7, 184.3)
- moved D32 33.1 mm to (239.1, 158.1)
- moved D4 33.1 mm to (95.9, 156.7)
- moved D6 33.1 mm to (107.0, 120.4)
- moved D16 33.1 mm to (135.4, 195.0)
- moved S6 33.1 mm to (108.2, 116.6)
- moved D10 33.1 mm to (131.9, 168.8)
- moved D33 33.1 mm to (233.6, 139.9)
- moved S11 33.1 mm to (138.7, 146.8)
- moved S24 33.1 mm to (286.0, 116.6)
- moved S13 33.1 mm to (150.7, 172.5)
- moved S26 33.1 mm to (272.6, 137.4)
- moved D30 33.1 mm to (251.2, 132.5)
- moved S2 33.1 mm to (82.1, 136.8)
- moved D35 33.1 mm to (239.9, 204.3)
- moved S10 33.1 mm to (133.1, 165.0)
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Routing:
- net P5: track 119.8 -> 128.5 mm, vias 9 -> 6
- net P16: track 145.3 -> 153.4 mm, vias 6 -> 5
- net P4: track 119.7 -> 127.4 mm, vias 9 -> 5
- net P6: track 141.0 -> 147.0 mm, vias 6 -> 7
- net P21: track 122.6 -> 127.0 mm, vias 8 -> 5
- net P20: track 138.9 -> 143.1 mm, vias 8 -> 5
- net P14: track 332.8 -> 335.2 mm
Other:
- outline, holes or cut-outs redrawn
